File: hw/IMU_ICM20948.kicad_sch (KiCad schematic)
At the start: 5 parts, among them U1 ICM-20948

Commit message: WIP
Parts:
- renumbered U1 to IMU1
Changed lines of the file:
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@@
 		(dnp no)
 		(fields_autoplaced yes)
-		(property "Reference" "U1"
+		(property "Reference" "IMU1"
 			(at 88.5033 72.39 0)
 			(effects
@@
 		)
 		(property "Description" "InvenSense 9-Axis Motion Sensor, Accelerometer, Gyroscope, Compass, I2C/SPI, QFN-24"
+			(at 86.36 54.61 0)
+			(effects
+				(font
+					(size 1.27 1.27)
+				)
+				(hide yes)
+			)
+		)
+		(property "Sim.Library" "/Users/msk-hq-nb-1221/pcb/multivibrator/magnitrometr/sim/models/icm20948_avg.lib"
+			(at 86.36 54.61 0)
+			(effects
+				(font
+					(size 1.27 1.27)
+				)
+				(hide yes)
+			)
+		)
+		(property "Sim.Name" "ICM20948_AVG"
+			(at 86.36 54.61 0)
+			(effects
+				(font
+					(size 1.27 1.27)
+				)
+				(hide yes)
+			)
+		)
+		(property "Sim.Device" "SUBCKT"
+			(at 86.36 54.61 0)
+			(effects
+				(font
+					(size 1.27 1.27)
+				)
+				(hide yes)
+			)
+		)
+		(property "Sim.Pins" "1=NC1 2=NC2 3=NC3 4=NC4 5=NC5 6=NC6 7=AUX_CL 8=VDDIO 9=SDOAD0 10=REGOUT 11=FSYNC 12=INT1 13=VDD 14=NC14 15=NC15 16=NC16 17=NC17 18=GND_A 19=RESV 20=GND_B 21=AUX_DA 22=nCS 23=SCL 24=SDA"
 			(at 86.36 54.61 0)
 			(effects
@@
 			(project ""
 				(path "/891cdf0c-b4c2-4f65-9c53-c267913f529d/ce5d4f46-d322-4fd2-88f9-a110a0579c5d"
-					(reference "U1")
+					(reference "IMU1")
 					(unit 1)
 				)
