File: hw/MCU_ESP32.kicad_sch (KiCad schematic)
At the start: 4 parts, among them U4 ESP32-WROOM-32

Commit message: WIP
Connections:
- net at R2.2: now also U4.30 (IO18); no longer U4.36 (IO22)
- net at R4.2: now also U4.31 (IO19); no longer U4.10 (IO25)
- net GPIO0: now reaches U4.25 (IO0)
- net EN: now reaches U4.3 (EN)
- net U0RXD: now reaches U4.34 (RXD0/IO3)
- net U0TXD: now reaches U4.35 (TXD0/IO1)
- no-connect marks 18 -> 14
Other:
- moved on the sheet: R2, R4
Changed lines of the file:
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@@
-	)
-	(no_connect
-		(at 116.84 67.31)
 	)
 	(no_connect
@@
 	)
 	(no_connect
-		(at 116.84 34.29)
-	)
-	(no_connect
 		(at 86.36 74.93)
 	)
 	(no_connect
-		(at 116.84 64.77)
-	)
-	(no_connect
 		(at 86.36 69.85)
 	)
@@
 	)
 	(no_connect
-		(at 86.36 34.29)
-	)
-	(no_connect
-		(at 116.84 41.91)
+		(at 116.84 77.47)
 	)
 	(no_connect
@@
 	)
 	(no_connect
+		(at 116.84 72.39)
+	)
+	(no_connect
 		(at 116.84 69.85)
 	)
-	(no_connect
-		(at 116.84 36.83)
+	(wire
+		(pts
+			(xy 119.38 36.83) (xy 116.84 36.83)
+		)
+		(stroke
+			(width 0)
+			(type default)
+		)
+	)
+	(wire
+		(pts
+			(xy 116.84 41.91) (xy 127 41.91)
+		)
+		(stroke
+			(width 0)
+			(type default)
+		)
 	)
 	(wire
@@
 	(wire
 		(pts
+			(xy 116.84 64.77) (xy 120.65 64.77)
+		)
+		(stroke
+			(width 0)
+			(type default)
+		)
+	)
+	(wire
+		(pts
 			(xy 101.6 26.67) (xy 101.6 29.21)
 		)
@@
 	(wire
 		(pts
+			(xy 81.28 34.29) (xy 86.36 34.29)
+		)
+		(stroke
+			(width 0)
+			(type default)
+		)
+	)
+	(wire
+		(pts
+			(xy 119.38 39.37) (xy 119.38 36.83)
+		)
+		(stroke
+			(width 0)
+			(type default)
+		)
+	)
+	(wire
+		(pts
 			(xy 116.84 85.09) (xy 121.92 85.09)
 		)
@@
 	(wire
 		(pts
-			(xy 133.35 72.39) (xy 129.54 72.39)
+			(xy 132.08 64.77) (xy 128.27 64.77)
 		)
 		(stroke
@@
 	(wire
 		(pts
+			(xy 127 39.37) (xy 119.38 39.37)
+		)
+		(stroke
+			(width 0)
+			(type default)
+		)
+	)
+	(wire
+		(pts
 			(xy 116.84 90.17) (xy 121.92 90.17)
 		)
@@
 	(wire
 		(pts
-			(xy 116.84 72.39) (xy 121.92 72.39)
+			(xy 116.84 67.31) (xy 120.65 67.31)
+		)
+		(stroke
+			(width 0)
+			(type default)
+		)
+	)
+	(wire
+		(pts
+			(xy 127 36.83) (xy 120.65 36.83)
 		)
 		(stroke
@@
 	(wire
 		(pts
-			(xy 116.84 77.47) (xy 121.92 77.47)
+			(xy 120.65 36.83) (xy 120.65 34.29)
+		)
+		(stroke
+			(width 0)
+			(type default)
+		)
+	)
+	(wire
+		(pts
+			(xy 120.65 34.29) (xy 116.84 34.29)
 		)
 		(stroke
@@
 	(wire
 		(pts
-			(xy 129.54 77.47) (xy 133.35 77.47)
+			(xy 128.27 67.31) (xy 132.08 67.31)
 		)
 		(stroke
@@
 		)
 	)
+	(hierarchical_label "GPIO0"
+		(shape passive)
+		(at 127 36.83 0)
+		(effects
+			(font
+				(size 1.27 1.27)
+			)
+			(justify left)
+		)
+	)
+	(hierarchical_label "U0RXD"
+		(shape passive)
+		(at 127 41.91 0)
+		(effects
+			(font
+				(size 1.27 1.27)
+			)
+			(justify left)
+		)
+	)
 	(hierarchical_label "M2_IN2"
 		(shape output)
@@
 	(hierarchical_label "SPI_SCLK"
 		(shape output)
-		(at 133.35 72.39 0)
+		(at 132.08 64.77 0)
 		(effects
 			(font
@@
 	(hierarchical_label "SPI_MISO"
 		(shape input)
-		(at 133.35 77.47 0)
+		(at 132.08 67.31 0)
+		(effects
+			(font
+				(size 1.27 1.27)
+			)
+			(justify left)
+		)
+	)
+	(hierarchical_label "U0TXD"
+		(shape passive)
+		(at 127 39.37 0)
 		(effects
 			(font
@@
 		)
 	)
+	(hierarchical_label "EN"
+		(shape passive)
+		(at 81.28 34.29 180)
+		(effects
+			(font
+				(size 1.27 1.27)
+			)
+			(justify right)
+		)
+	)
 	(hierarchical_label "ENC1_A"
 		(shape input)
@@
 	(symbol
 		(lib_id "Device:R")
-		(at 125.73 72.39 270)
+		(at 124.46 64.77 270)
 		(unit 1)
 		(exclude_from_sim no)
@@
 		(dnp no)
 		(property "Reference" "R2"
-			(at 125.476 70.104 90)
+			(at 128.524 64.008 90)
 			(effects
 				(font
@@
 		)
 		(property "Value" "33"
-			(at 125.476 72.39 90)
+			(at 124.206 64.77 90)
 			(effects
 				(font
@@
 		)
 		(property "Footprint" "Resistor_SMD:R_0603_1608Metric"
-			(at 125.73 70.612 90)
+			(at 124.46 62.992 90)
 			(effects
 				(font
@@
 		)
 		(property "Datasheet" "~"
-			(at 125.73 72.39 0)
+			(at 124.46 64.77 0)
 			(effects
 				(font
@@
 		)
 		(property "Description" "Resistor"
-			(at 125.73 72.39 0)
+			(at 124.46 64.77 0)
 			(effects
 				(font
@@
 	(symbol
 		(lib_id "Device:R")
-		(at 125.73 77.47 270)
+		(at 124.46 67.31 270)
 		(unit 1)
 		(exclude_from_sim no)
@@
 		(dnp no)
 		(property "Reference" "R4"
-			(at 125.73 79.502 90)
+			(at 124.46 69.342 90)
 			(effects
 				(font
@@
 		)
 		(property "Value" "33"
-			(at 125.73 77.47 90)
+			(at 124.46 67.31 90)
 			(effects
 				(font
@@
 		)
 		(property "Footprint" "Resistor_SMD:R_0603_1608Metric"
-			(at 125.73 75.692 90)
+			(at 124.46 65.532 90)
 			(effects
 				(font
@@
 		)
 		(property "Datasheet" "~"
-			(at 125.73 77.47 0)
+			(at 124.46 67.31 0)
 			(effects
 				(font
@@
 		)
 		(property "Description" "Resistor"
-			(at 125.73 77.47 0)
+			(at 124.46 67.31 0)
 			(effects
 				(font
@@
 		(at 101.6 64.77 0)
 		(unit 1)
-		(exclude_from_sim no)
+		(exclude_from_sim yes)
 		(in_bom yes)
 		(on_board yes)
