File: hw/power.kicad_sch (KiCad schematic)
At the start: 18 parts, among them J2 7.4V, U2 TPS62162DSG, U3 TLV70018_SOT23-5

Commit message: Add tests
Parts:
- renumbered J2 to POWER_SOURCE1
Changed lines of the file:
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@@
 		(at 33.02 38.1 0)
 		(unit 1)
-		(exclude_from_sim no)
+		(exclude_from_sim yes)
 		(in_bom yes)
 		(on_board yes)
@@
 		(at 43.18 81.28 0)
 		(unit 1)
-		(exclude_from_sim no)
+		(exclude_from_sim yes)
 		(in_bom yes)
 		(on_board yes)
@@
 		(at 83.82 33.02 0)
 		(unit 1)
-		(exclude_from_sim no)
+		(exclude_from_sim yes)
 		(in_bom yes)
 		(on_board yes)
@@
 		(mirror y)
 		(unit 1)
-		(exclude_from_sim no)
-		(in_bom yes)
-		(on_board yes)
-		(dnp no)
-		(property "Reference" "J2"
+		(exclude_from_sim yes)
+		(in_bom yes)
+		(on_board yes)
+		(dnp no)
+		(property "Reference" "POWER_SOURCE1"
 			(at 157.48 27.9399 0)
 			(effects
@@
 			(project ""
 				(path "/891cdf0c-b4c2-4f65-9c53-c267913f529d/32dcc24e-8308-45ed-b18e-b6bb77f40255"
-					(reference "J2")
-					(unit 1)
-				)
+					(reference "POWER_SOURCE1")
+					(unit 1)
+				)

Commit message: WIP
Parts:
- added C_GATE_SOFT1: 47n, Capacitor_SMD:C_0805_2012Metric, symbol Device:C
- added GROUND_POINT1: GND, TestPoint:TestPoint_Pad_1.0x1.0mm, symbol Connector:TestPoint
- added LOGIC_POINT1: VLOGIC, TestPoint:TestPoint_Pad_1.0x1.0mm, symbol Connector:TestPoint
- added MOTOR_POINT1: VMOTOR, TestPoint:TestPoint_Pad_1.0x1.0mm, symbol Connector:TestPoint
- added POWER_POLYFUSE1: 2A, Fuse:Fuse_Bourns_MF-RHT200, symbol Device:Polyfuse_Small
- added Q1: Q_PMOS_GSD, Package_TO_SOT_SMD:SOT-23, symbol Transistor_FET:Q_PMOS_GSD
- added R_GATE_PULL1: 100k, Resistor_SMD:R_0612_1632Metric, symbol Device:R
- added SW1: SW_SPST, Button_Switch_SMD:SW_SPDT_PCM12, symbol Switch:SW_SPST
- added V1: 7.4, symbol Simulation_SPICE:VDC
- added VIO18_POINT1: VIO18, TestPoint:TestPoint_Pad_1.0x1.0mm, symbol Connector:TestPoint
- renumbered U3 to 3V3_TO_1V8, U2 to 7V4_TO_3V3
Connections:
- net GND: now also 7V4_TO_3V3.5 (FB), C_3V3_dec1.2, C_3V3_dec2.2, C_GATE_SOFT1.1, GROUND_POINT1.1, R_GATE_PULL1.1, SW1.1 (A), V1.2
- net VIO18: now also VIO18_POINT1.1
- net VLOGIC: now also LOGIC_POINT1.1
- net VLOGIC_MPU: now also C_3V3_dec1.1, FB1.2; no longer C_3V3_dec1.2
- net VLOGIC_RF: now also C_3V3_dec2.1, FB2.2; no longer C_3V3_dec2.2
- net VMOTOR: now also MOTOR_POINT1.1, Q1.3 (D), V1.1; no longer POWER_SOURCE1.1 (Pin_1)
- new net: C_GATE_SOFT1.2, Q1.1 (G), R_GATE_PULL1.2, SW1.2 (B)
- new net: POWER_POLYFUSE1.1, Q1.2 (S)
- new net: POWER_POLYFUSE1.2, POWER_SOURCE1.1 (Pin_1)
- no-connect marks 1 -> 0
Other:
- moved on the sheet: C_3V3_dec1, C_3V3_dec2, POWER_SOURCE1
